Commit message: mapping algo added

File: rotf_control/urdf/model.urdf (robot description, URDF)
Before this commit: robot diff_bot, 4 links, 3 joints
Links:
- link base_link: mass 50 -> 15; geometry collision box size=.5 .3 .1; collision sphere radius=0.05
- link left_wheel: mass 2.5 -> 1; geometry collision cylinder length=0.03 radius=0.1; visual cylinder length=0.03 radius=0.1
- link right_wheel: mass 2.5 -> 1; geometry collision cylinder length=0.03 radius=0.1; visual cylinder length=0.03 radius=0.1

Commit message: updates

File: rotf_control/urdf/model.urdf (robot description, URDF)
Before this commit: robot diff_bot, 4 links, 3 joints
Joints:
- joint laser_joint: origin xyz=0 0 0.080 rpy=0 0 0 -> xyz=0 0 0.12 rpy=0 0 0
